File: USB_PCIE_BOARD_POWER.kicad_sch (KiCad schematic)
At the start: 0 parts

Commit message: Added power conversion circuits
Parts:
- added C45, C46: 6.8uF, Capacitor_SMD:C_1206_3216Metric_Pad1.33x1.80mm_HandSolder, symbol 0_Custom:CAP_1206_6.8uF_35V
- added C47: 22uF, Capacitor_SMD:CP_Elec_6.3x5.9, symbol 0_Custom:CAP_POL_SMD_22uF
- added C48: 180uF, Capacitor_SMD:CP_Elec_8x10.5, symbol 0_Custom:CAP_POL_SMD_180uF
- added C49: 10nF, Capacitor_SMD:C_1206_3216Metric_Pad1.33x1.80mm_HandSolder, symbol 0_Custom:CAP_1206_10nF_50V
- added C50, C57, C59: 0.1uF, Capacitor_SMD:C_0603_1608Metric_Pad1.08x0.95mm_HandSolder, symbol 0_Custom:CAP_0603_0.1uF_50V
- added C51, C56: 10uF, Capacitor_SMD:C_1206_3216Metric_Pad1.33x1.80mm_HandSolder, symbol 0_Custom:CAP_1206_10uF_25V
- added C52: 1.8nF, Capacitor_SMD:C_0402_1005Metric_Pad0.74x0.62mm_HandSolder, symbol 0_Custom:CAP_0402_1.8nF_50V
- added C53: 47pF, Capacitor_SMD:C_0402_1005Metric_Pad0.74x0.62mm_HandSolder, symbol 0_Custom:CAP_0402_47pF_50V
- added C54, C55: 100uF, Capacitor_SMD:C_1210_3225Metric_Pad1.33x2.70mm_HandSolder, symbol 0_Custom:CAP_1210_100uF_10V
- added C58, C60, C61: 22uF, Capacitor_SMD:C_0603_1608Metric_Pad1.08x0.95mm_HandSolder, symbol 0_Custom:CAP_0603_22uF_6.3V
- added C62, C63, C66, C69, C74, C75: 1uF, Capacitor_SMD:C_0603_1608Metric_Pad1.08x0.95mm_HandSolder, symbol 0_Custom:CAP_0603_1uF_25V
- added C64, C67, C70, C71: 10uF, Capacitor_SMD:C_0805_2012Metric_Pad1.18x1.45mm_HandSolder, symbol 0_Custom:CAP_0805_10uF_16V
- added C65, C68, C72, C73: 150uF, Capacitor_SMD:CP_Elec_8x6.9, symbol 0_Custom:CAP_POL_SMD_150uF
- added D2: B560C-13-F, Diode_SMD:D_SMC_Handsoldering, symbol 0_Custom:B560C-13-F_D
- added D3: RB081L-20, PCM_Diode_SMD_AKL:D_SMA, symbol PCM_Diode_Schottky_AKL:RB081L-20
- added D4, D5: RBR2MM30BTR, Diode_SMD:D_SOD-123F, symbol 0_Custom:RBR2MM30BTR_D
- added D6: B320A-13-F, Diode_SMD:D_SMA, symbol 0_Custom:B320A-13-F_D
- added F1: 32V/3.15A, Fuse:Fuse_0603_1608Metric_Pad1.05x0.95mm_HandSolder, symbol 0_Custom:FUSE_0603_32V/3.15A
- added L1: 3.9uH, 0_Custom:IND_BOURNS_SRU8043, symbol 0_Custom:IND_SRU8043-3R9Y_3.9uH
- added L2: 1uH, 0_Custom:IND_SPM6530T-1R0M120, symbol 0_Custom:IND_SPM6530T-1R0M120_1uH
- added L3: 1.5uH, Inductor_SMD:L_1008_2520Metric_Pad1.43x2.20mm_HandSolder, symbol 0_Custom:IND_1008_1.5uH
- added Q1: 2SA1576AT106R, 0_Custom:SOT-323_SC-70, symbol 0_Custom:2SA1576AT106R_Q
- added Q2: 2SC4081T106R, 0_Custom:SOT-323_SC-70, symbol 0_Custom:2SC4081T106R_Q
- added Q4: DMT6016LSS-13, PCM_SparkFun-Semiconductor-Standard:SO-8, symbol 0_Custom:DMT6016LSS-13_Q
- added Q5: SI4134DY-T1-GE3, PCM_Package_SO_AKL:SO-8_3.9x4.9mm_P1.27mm, symbol 0_Custom:SI4134DY-T1-GE3_Q
- added R16, R23, R27, R28, R29, R30: 10K, Resistor_SMD:R_0603_1608Metric_Pad0.98x0.95mm_HandSolder, symbol 0_Custom:RES_0603_10K
- added R17, R26, R31: 0R, Resistor_SMD:R_1206_3216Metric_Pad1.30x1.75mm_HandSolder, symbol 0_Custom:RES_1206_0R
- added R18: 47K, Resistor_SMD:R_0603_1608Metric_Pad0.98x0.95mm_HandSolder, symbol 0_Custom:RES_0603_47K
- added R19: 11K, Resistor_SMD:R_0402_1005Metric_Pad0.72x0.64mm_HandSolder, symbol 0_Custom:RES_0402_11K_50V
- added R20: 17.4K, Resistor_SMD:R_0402_1005Metric_Pad0.72x0.64mm_HandSolder, symbol 0_Custom:RES_0402_17.4K
- added R21: 34.8K, Resistor_SMD:R_0402_1005Metric_Pad0.72x0.64mm_HandSolder, symbol 0_Custom:RES_0402_34.8K_50V
- added R22: 1M, Resistor_SMD:R_0603_1608Metric_Pad0.98x0.95mm_HandSolder, symbol 0_Custom:RES_0603_1M
- added R24: 100K, Resistor_SMD:R_0603_1608Metric_Pad0.98x0.95mm_HandSolder, symbol 0_Custom:RES_0603_100K
- added R25: 133K, Resistor_SMD:R_0603_1608Metric_Pad0.98x0.95mm_HandSolder, symbol 0_Custom:RES_0603_133K
- added TP4, TP5, TP6, TP7: D0.5mm, TestPoint:TestPoint_THTPad_1.0x1.0mm_Drill0.5mm, symbol Connector:TestPoint
- added U10, U11, U8, U9: AP2191SG-13, Package_SO:HSOP-8-1EP_3.9x4.9mm_P1.27mm_EP2.3x2.3mm, symbol 0_Custom:AP2191SG-13_PSW
- added U3: LM22678TJ-5.0/NOPB, Package_TO_SOT_SMD:TO-263-7_TabPin8, symbol 0_Custom:LM22678TJ-5.0/NOPB
- added U4: LTC3872ETS8-TRPBF, Package_TO_SOT_SMD:TSOT-23-8, symbol 0_Custom:LTC3872ETS8-TRPBF
- added U5: RT5762CHGH6F, Package_TO_SOT_SMD:SOT-563, symbol 0_Custom:RT5762CHGH6F
- added U6: 641737-1, 0_Custom:641737-1_TYC, symbol 0_Custom:641737-1_ATX_4-POS
- added U7: AP7215-33YG-13, Package_TO_SOT_SMD:SOT-89-3, symbol 0_Custom:AP7215-33YG-13_REG
Connections:
- new net: R19.2, R21.1, U4.3 (VFB)
- new net: D4.1 (K), D5.1 (K), R17.1
- new net: C60.1, C61.1, L3.2, R24.1, R31.2, TP7.1
- new net: C60.2, R24.2, R25.1, U5.1 (FB)
- new net: Q2.1 (B), R23.1
- new net: Q2.2 (C), R18.1
- new net: C50.1, C51.1, F1.1, U6.1 (+12V)
- new net: C53.2, R20.2, U4.2 (ITH)
- new net: C48.1, D3.2 (A), L1.2, U3.6 (FB)
- new net: Q1.2 (E), Q4.4, R16.1
- new net: C52.2, R20.1
- new net: L3.1, U5.4 (SW)
- new net: D6.2 (A), L2.2, Q5.5 (D), Q5.6 (D), Q5.7 (D), Q5.8 (D), U4.8 (SW)
- new net: Q1.1 (B), R18.2
- new net: C57.1, R22.1
- new net: C63.1, R26.2, TP5.1, U7.3 (VO)
- new net: D5.2 (A), F1.2
- new net: C49.1, U3.3 (BOOT)
- new net: C49.2, D2.1 (K), L1.1, U3.1 (SW)
- new net: Q5.4 (G), U4.5 (NGATE)
- new net +12V: D4.2 (A)
- new net +12V_IN: C45.1, C46.1, C47.1, Q1.3 (C), R17.2, U3.2 (VIN), U3.7 (EN)
- new net +1V05: R31.1, TP6.1
- new net +3V3: Q4.1, Q4.2, Q4.3, R23.2
- new net +3V3_DUAL: R26.1, R27.1, R28.1, R29.1, R30.1, TP4.1
- new net +3V3_SW: C56.1, C58.1, C59.1, L2.1, Q4.5, Q4.6, Q4.7, Q4.8, R22.2, U4.1 (IPRG), U4.6 (VIN), U5.3 (VIN), U5.5 (EN)
- new net +5V: C54.1, C55.1, C62.1, C66.1, C69.1, C74.1, C75.1, D3.1 (K), D6.1 (K), R21.2, U10.2 (IN), U10.3 (IN), U11.2 (IN), U11.3 (IN), U7.2 (VI), U8.2 (IN), U8.3 (IN), U9.2 (IN), U9.3 (IN)
- new net GND: C45.2, C46.2, C47.2, C48.2, C50.2, C51.2, C52.1, C53.1, C54.2, C55.2, C56.2, C57.2, C58.2, C59.2, C61.2, C62.2, C63.2, C64.2, C65.2, C66.2, C67.2, C68.2, C69.2, C70.2, C71.2, C72.2, C73.2, C74.2, C75.2, D2.2 (A), Q2.3 (E), Q5.1 (S), Q5.2 (S), Q5.3 (S), R16.2, R19.1, R25.2, U10.1 (GND), U11.1 (GND), U3.4 (GND), U3.8 (GND), U4.4 (GND), U5.2 (GND), U6.2 (COM), U6.3 (COM), U7.1 (GND), U8.1 (GND), U9.1 (GND)
- new net OCI3B: R28.2, R30.2, U11.5 (~{FLG}), U9.5 (~{FLG})
- new net OCI4B: R27.2, R29.2, U10.5 (~{FLG}), U8.5 (~{FLG})
- new net PPON3: U11.4 (EN), U9.4 (EN)
- new net PPON4: U10.4 (EN), U8.4 (EN)
- new net VCCCH1: C71.1, C73.1, U11.6 (OUT), U11.7 (OUT), U11.8 (NC)
- new net VCCCH2: C70.1, C72.1, U10.6 (OUT), U10.7 (OUT), U10.8 (NC)
- new net VCCCH3: C67.1, C68.1, U9.6 (OUT), U9.7 (OUT), U9.8 (NC)
- new net VCCCH4: C64.1, C65.1, U8.6 (OUT), U8.7 (OUT), U8.8 (NC)
- no-connect marks 0 -> 1

Commit message: Fix changes suggested by Claude review; added schematic and netlist to document folder
Connections:
- net +12V_IN: no longer U3.7 (EN)
- net OCI2B: now also R29.2, U10.5 (~{FLG})
- net OCI3B: no longer R30.2, U11.5 (~{FLG})
- net OCI4B: no longer R29.2, U10.5 (~{FLG})
- net PPON1: now also U11.4 (EN)
- net PPON2: now also U10.4 (EN)
- net PPON3: no longer U11.4 (EN)
- net PPON4: no longer U10.4 (EN)
- net at C57.1, R22.1: now also U4.7 (RUN/SS)
- new net OCI1B: R30.2, U11.5 (~{FLG})
- no-connect marks 1 -> 2
Changed lines of the file:
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@@
 	)
 	(junction
+		(at 241.3 182.88)
+		(diameter 0)
+		(color 0 0 0 0)
+	)
+	(junction
 		(at 450.85 307.34)
 		(diameter 0)
@@
 	)
 	(junction
-		(at 241.3 121.92)
-		(diameter 0)
-		(color 0 0 0 0)
-	)
-	(junction
 		(at 501.65 228.6)
 		(diameter 0)
@@
 	)
 	(no_connect
+		(at 243.84 127)
+	)
+	(no_connect
 		(at 88.9 121.92)
 	)
@@
 	(wire
 		(pts
-			(xy 241.3 121.92) (xy 243.84 121.92)
+			(xy 228.6 121.92) (xy 243.84 121.92)
 		)
 		(stroke
@@
 	(wire
 		(pts
+			(xy 241.3 182.88) (xy 241.3 199.39)
+		)
+		(stroke
+			(width 0)
+			(type default)
+		)
+	)
+	(wire
+		(pts
 			(xy 203.2 143.51) (xy 215.9 143.51)
 		)
@@
 	(wire
 		(pts
-			(xy 232.41 182.88) (xy 245.11 182.88)
+			(xy 232.41 182.88) (xy 241.3 182.88)
 		)
 		(stroke
@@
 	(wire
 		(pts
-			(xy 228.6 121.92) (xy 241.3 121.92)
-		)
-		(stroke
-			(width 0)
-			(type default)
-		)
-	)
-	(wire
-		(pts
 			(xy 520.7 307.34) (xy 520.7 317.5)
 		)
@@
 	(wire
 		(pts
+			(xy 241.3 182.88) (xy 245.11 182.88)
+		)
+		(stroke
+			(width 0)
+			(type default)
+		)
+	)
+	(wire
+		(pts
 			(xy 450.85 243.84) (xy 459.74 243.84)
 		)
@@
 	(wire
 		(pts
-			(xy 241.3 127) (xy 241.3 121.92)
-		)
-		(stroke
-			(width 0)
-			(type default)
-		)
-	)
-	(wire
-		(pts
 			(xy 482.6 292.1) (xy 495.3 292.1)
 		)
@@
 	(wire
 		(pts
-			(xy 243.84 127) (xy 241.3 127)
-		)
-		(stroke
-			(width 0)
-			(type default)
-		)
-	)
-	(wire
-		(pts
 			(xy 501.65 292.1) (xy 501.65 285.75)
 		)
@@
 		)
 	)
-	(global_label "OCI2B"
-		(shape output)
-		(at 438.15 257.81 0)
-		(fields_autoplaced yes)
-		(effects
-			(font
-				(size 1.27 1.27)
-			)
-			(justify left)
-		)
-		(property "Intersheetrefs" "${INTERSHEET_REFS}"
-			(at 446.82 257.81 0)
-			(hide yes)
-			(show_name no)
-			(do_not_autoplace no)
-			(effects
-				(font
-					(size 1.27 1.27)
-				)
-				(justify left)
-			)
-		)
-	)
-	(global_label "OCI3B"
+	(global_label "OCI1B"
 		(shape output)
 		(at 444.5 307.34 180)
@@
 		)
 	)
-	(global_label "OCI4B"
-		(shape output)
-		(at 444.5 243.84 180)
-		(fields_autoplaced yes)
-		(effects
-			(font
-				(size 1.27 1.27)
-			)
-			(justify right)
-		)
-		(property "Intersheetrefs" "${INTERSHEET_REFS}"
-			(at 435.83 243.84 0)
-			(hide yes)
-			(show_name no)
-			(do_not_autoplace no)
-			(effects
-				(font
-					(size 1.27 1.27)
-				)
-				(justify right)
-			)
-		)
-	)
 	(global_label "PPON2"
 		(shape input)
-		(at 438.15 264.16 0)
+		(at 444.5 238.76 180)
 		(fields_autoplaced yes)
 		(effects
@@
 				(size 1.27 1.27)
 			)
-			(justify left)
+			(justify right)
 		)
 		(property "Intersheetrefs" "${INTERSHEET_REFS}"
-			(at 447.5457 264.16 0)
+			(at 435.1043 238.76 0)
 			(hide yes)
 			(show_name no)
@@
 					(size 1.27 1.27)
 				)
-				(justify left)
+				(justify right)
 			)
 		)
@@
 	(global_label "PPON4"
 		(shape input)
-		(at 444.5 238.76 180)
-		(fields_autoplaced yes)
-		(effects
-			(font
-				(size 1.27 1.27)
-			)
-			(justify right)
-		)
-		(property "Intersheetrefs" "${INTERSHEET_REFS}"
-			(at 435.1043 238.76 0)
-			(hide yes)
-			(show_name no)
-			(do_not_autoplace no)
-			(effects
-				(font
-					(size 1.27 1.27)
-				)
-				(justify right)
-			)
-		)
-	)
-	(global_label "PPON4"
-		(shape input)
 		(at 444.5 111.76 180)
 		(fields_autoplaced yes)
@@
 	(global_label "OCI2B"
 		(shape output)
-		(at 438.15 260.35 0)
+		(at 444.5 243.84 180)
 		(fields_autoplaced yes)
 		(effects
@@
 				(size 1.27 1.27)
 			)
-			(justify left)
+			(justify right)
 		)
 		(property "Intersheetrefs" "${INTERSHEET_REFS}"
-			(at 446.82 260.35 0)
+			(at 435.83 243.84 0)
 			(hide yes)
 			(show_name no)
@@
 					(size 1.27 1.27)
 				)
-				(justify left)
+				(justify right)
 			)
 		)
 	)
-	(global_label "PPON3"
+	(global_label "PPON1"
 		(shape input)
 		(at 444.5 302.26 180)
@@
 			)
 		)
-	)
-	(global_label "PPON1"
-		(shape input)
-		(at 438.15 266.7 0)
-		(fields_autoplaced yes)
-		(effects
-			(font
-				(size 1.27 1.27)
-			)
-			(justify left)
-		)
-		(property "Intersheetrefs" "${INTERSHEET_REFS}"
-			(at 447.5457 266.7 0)
-			(hide yes)
-			(show_name no)
-			(do_not_autoplace no)
-			(effects
-				(font
-					(size 1.27 1.27)
-				)
-				(justify left)
-			)
-		)

Commit message: Add indicator LEDs and run ERC
Parts:
- added D10, D7, D8, D9: LED_0805_WHITE, LED_SMD:LED_0805_2012Metric_Pad1.15x1.40mm_HandSolder, symbol 0_Custom:LED_0805_WHITE
- added D11, D12, D13: LED_0805_BLUE, LED_SMD:LED_0805_2012Metric_Pad1.15x1.40mm_HandSolder, symbol 0_Custom:LED_0805_BLUE
- added D14, D15: LED_0805_YELLOW, LED_SMD:LED_0805_2012Metric_Pad1.15x1.40mm_HandSolder, symbol 0_Custom:LED_0805_YELLOW
- added R32, R33, R34, R35, R36, R37, R38, R39: 1K, Resistor_SMD:R_0603_1608Metric_Pad0.98x0.95mm_HandSolder, symbol 0_Custom:RES_0603_1K
- added R40: 10K, Resistor_SMD:R_0603_1608Metric_Pad0.98x0.95mm_HandSolder, symbol 0_Custom:RES_0603_10K
Connections:
- net +12V_IN: now also D15.2 (A)
- net +1V05: now also D11.2 (A)
- net +3V3_DUAL: now also D13.2 (A)
- net +3V3_SW: now also D14.2 (A)
- net +5V: now also D12.2 (A)
- net GND: now also R32.2, R33.2, R34.2, R35.2, R36.2, R37.2, R38.2, R39.2, R40.2
- net VCCCH1: now also D10.2 (A)
- net VCCCH2: now also D9.2 (A)
- net VCCCH3: now also D7.2 (A)
- net VCCCH4: now also D8.2 (A)
- new net: D11.1 (K), R36.1
- new net: D15.1 (K), R40.1
- new net: D10.1 (K), R35.1
- new net: D7.1 (K), R32.1
- new net: D8.1 (K), R33.1
- new net: D12.1 (K), R37.1
- new net: D9.1 (K), R34.1
- new net: D13.1 (K), R38.1
- new net: D14.1 (K), R39.1

Commit message: Place all components except host chip decoupling caps and the crystal circuit.
Parts:
- D3: value RB081L-20 -> RSX501LAM20TR; footprint PCM_Diode_SMD_AKL:D_SMA -> Diode_SMD:D_SOD-128; symbol PCM_Diode_Schottky_AKL:RB081L-20 -> 0_Custom:RSX501LAM20TR_D; DigiKey Part # (none) -> RSX501LAM20CT-ND; LCSC Part # (none) -> C253526; Manufacturer (none) -> ROHM; Manufacturer Part # (none) -> RSX501LAM20TR; Package (none) -> SOD-128
- Q5: footprint PCM_Package_SO_AKL:SO-8_3.9x4.9mm_P1.27mm -> 0_Custom:SO-8_3.9x4.9mm_P1.27mm
- TP4, TP5, TP6, TP7: value D0.5mm -> TestPoint
- U10, U11, U8, U9: footprint Package_SO:HSOP-8-1EP_3.9x4.9mm_P1.27mm_EP2.3x2.3mm -> 0_Custom:HSOP-8-1EP_3.9x4.9mm_P1.27mm_EP2.3x2.3mm
Other:
- moved on the sheet: D3
