File: USB_PCIE_Board.kicad_sch (KiCad schematic)
At the start: 0 parts

Commit message: Populated host schematic and power caps
Parts:
- added C1, C10, C11, C12, C13, C14, C15, C16, C17, C2, C3, C4, C5, C6, C7, C8, C9: 0.01uF, Capacitor_SMD:C_0402_1005Metric_Pad0.74x0.62mm_HandSolder, symbol 0_Custom:CAP_0402_0.01uF
- added C18, C19, C20, C21, C22, C23, C24, C25, C26, C27, C29: 0.1uF, Capacitor_SMD:C_0402_1005Metric_Pad0.74x0.62mm_HandSolder, symbol 0_Custom:CAP_0402_0.1uF_16V
- added C28: 1uF, Capacitor_SMD:C_0603_1608Metric_Pad1.08x0.95mm_HandSolder, symbol 0_Custom:CAP_0603_1uF_25V
- added C30, C31: 8pF, Capacitor_SMD:C_0402_1005Metric_Pad0.74x0.62mm_HandSolder, symbol 0_Custom:CAP_0402_8pF_50V
- added D1: 1SS294,LF, PCM_Package_TO_SOT_SMD_AKL:SC-59, symbol 0_Custom:1SS294,LF_D
- added J1: Bus_PCI_Express_x1, Connector_PCBEdge:BUS_PCIexpress_x1, symbol 0_Custom:Bus_PCI_Express_x1
- added J2, J3, J4, J5: GSB4116341HR, 0_Custom:AMPHENOL_GSB4116341HR, symbol 0_Custom:GSB4116341HR
- added R1: 0R, Resistor_SMD:R_0603_1608Metric_Pad0.98x0.95mm_HandSolder, symbol 0_Custom:RES_0603_0R
- added R2, R3, R5, R6, R7: 10K, Resistor_SMD:R_0603_1608Metric_Pad0.98x0.95mm_HandSolder, symbol 0_Custom:RES_0603_10K
- added R4: 100K, Resistor_SMD:R_0603_1608Metric_Pad0.98x0.95mm_HandSolder, symbol 0_Custom:RES_0603_100K
- added R8: 1.6K, Resistor_SMD:R_0402_1005Metric_Pad0.72x0.64mm_HandSolder, symbol 0_Custom:RES_0603_1.6K
- added R9: 680R, Resistor_SMD:R_0402_1005Metric_Pad0.72x0.64mm_HandSolder, symbol 0_Custom:RES_0402_680R
- added TP1, TP2: D0.5mm, TestPoint:TestPoint_THTPad_1.0x1.0mm_Drill0.5mm, symbol Connector:TestPoint
- added U1: UPD720201K8-711-BAC-A, 0_Custom:QFN68_8X8_REN-M, symbol 0_Custom:UPD720201K8-711-BAC-A
- added U2: MX25L4006EM1I-12G, Package_SO:HSOP-8-1EP_3.9x4.9mm_P1.27mm_EP2.3x2.3mm, symbol 0_Custom:MX25L4006EM1I-12G_FLASH
- added X1: CS14522-24M, Crystal:Crystal_SMD_3225-4Pin_3.2x2.5mm_HandSoldering, symbol 0_Custom:CS14522-24M_XTAL
Connections:
- new net: TP1.1, U1.13 (PECREQB)
- new net: TP2.1, U1.1 (SMIB)
- new net: C31.1, R9.1, X1.3
- new net: R6.2, U2.3 (~{WP})
- new net +1V05: C10.2, C11.2, C12.2, C13.2, C14.2, C15.2, C20.1, C21.1, C22.1, C23.1, C7.2, C8.2, C9.2, U1.12 (VDD10), U1.28 (VDD10), U1.37 (VDD10), U1.43 (VDD10), U1.46 (VDD10), U1.54 (VDD10), U1.60 (VDD10), U1.63 (VDD10), U1.9 (VDD10)
- new net +3V3A: C16.2, C17.2, C24.1, C25.1, U1.32 (AVDD33), U1.6 (AVDD33)
- new net +3V3_DUAL: C1.2, C18.1, C19.1, C2.2, C29.1, C3.2, C4.2, C5.2, C6.2, D1.3 (K), R2.1, R3.1, R5.1, R6.1, R7.1, U1.15 (VDD33), U1.29 (VDD33), U1.40 (VDD33), U1.49 (VDD33), U1.57 (VDD33), U1.66 (VDD33), U2.7 (~{HOLD}), U2.8 (VCC)
- new net GND: C1.1, C10.1, C11.1, C12.1, C13.1, C14.1, C15.1, C16.1, C17.1, C18.2, C19.2, C2.1, C20.2, C21.2, C22.2, C23.2, C24.2, C25.2, C28.2, C29.2, C3.1, C30.2, C31.2, C4.1, C5.1, C6.1, C7.1, C8.1, C9.1, R4.2, R8.1, U1.34 (IC(L)), U1.69 (GND), U2.4 (GND), X1.2, X1.4
- new net PECLKN: U1.5 (PECLKN)
- new net PECLKP: U1.4 (PECLKP)
- new net PERSTB: U1.2 (PERSTB)
- new net PERXN: U1.11 (PERXN)
- new net PERXP: U1.10 (PERXP)
- new net PETXN: C27.2, J1.B15 (PETn0)
- new net PETXN_H: C27.1, U1.8 (PETXN)
- new net PETXP: C26.1, J1.B14 (PETp0)
- new net PETXP_H: C26.2, U1.7 (PETXP)
- new net PEWAKEB: J1.B11 (~{WAKE}), R1.1
- new net PEWAKEB_H: R1.2, U1.3 (PEWAKEB)
- new net PONRSTB: C28.1, D1.1 (A), R2.2, U1.14 (PONRSTB)
- new net RREF: R8.2, U1.33 (RREF)
- new net SPICSB: R3.2, U1.17 (SPICSB), U2.1 (~{CS})
- new net SPISCK: R4.1, U1.18 (SPISCK), U2.6 (SCLK)
- new net SPISI: R7.2, U1.19 (SPISI), U2.5 (SI)
- new net SPISO: R5.2, U1.16 (SPISO), U2.2 (SO)
- new net XT1: C30.1, U1.31 (XT1), X1.1
- new net XT2: R9.2, U1.30 (XT2)
Other:
- added sheet POWER (USB_PCIE_BOARD_POWER.kicad_sch)
- title: (none) -> USB PCIE Expansion Card Board

Commit message: Populated all connections and components in the host controller page
Parts:
- added C32, C34, C35: 10uF, Capacitor_SMD:C_0805_2012Metric_Pad1.18x1.45mm_HandSolder, symbol 0_Custom:CAP_0805_10uF_16V
- added C33, C36: 0.1uF, Capacitor_SMD:C_0603_1608Metric_Pad1.08x0.95mm_HandSolder, symbol 0_Custom:CAP_0603_0.1uF_50V
- added C37, C38, C39, C40, C41, C42, C43, C44: 0.1uF, Capacitor_SMD:C_0402_1005Metric_Pad0.74x0.62mm_HandSolder, symbol 0_Custom:CAP_0402_0.1uF_16V
- added FB1, FB2, FB3, FB4, FB5: BLM21PG600SN1D, 0_Custom:Ferrite_0805_2012Metric_BigPads, symbol 0_Custom:BLM21PG600SN1D_FB
- added R10, R11: 0R, Resistor_SMD:R_1206_3216Metric_Pad1.30x1.75mm_HandSolder, symbol 0_Custom:RES_1206_0R
- added R12, R13, R14, R15: 0R, Resistor_SMD:R_0603_1608Metric_Pad0.98x0.95mm_HandSolder, symbol 0_Custom:RES_0603_0R
- added TP3: D0.5mm, TestPoint:TestPoint_THTPad_1.0x1.0mm_Drill0.5mm, symbol Connector:TestPoint
Connections:
- net +3V3A: now also C32.1, FB1.2
- net +3V3_DUAL: now also FB1.1
- net GND: now also J1.A12 (GND), J1.A15 (GND), J1.A18 (GND), J1.A4 (GND), J1.B13 (GND), J1.B16 (GND), J1.B18 (GND), J1.B4 (GND), J1.B7 (GND), J2.4 (GND), J2.7 (GND_DRAIN), J3.4 (GND), J3.7 (GND_DRAIN), J4.4 (GND), J4.7 (GND_DRAIN), J5.4 (GND), J5.7 (GND_DRAIN), C32.2, C33.2, C34.2, C35.2, C36.2, R12.1, R13.1, R14.1, R15.1
- net PECLKN: now also J1.A14 (REFCLK-)
- net PECLKP: now also J1.A13 (REFCLK+)
- net PERSTB: now also J1.A11 (~{PERST})
- net PERXN: now also J1.B15 (PETn0)
- net PERXP: now also J1.B14 (PETp0)
- net PETXN: now also J1.A17 (PERn0); no longer J1.B15 (PETn0)
- net PETXP: now also J1.A16 (PERp0); no longer J1.B14 (PETp0)
- net at J2.1 (VBUS): now also FB2.2
- net U2DM4: now reaches J2.2 (D-)
- net U2DM4: now also U1.68 (U2DM4)
- net U2DP4: now reaches J2.3 (D+)
- net U2DP4: now also U1.67 (U2DP4)
- net U3RXDN4: now reaches J2.5 (SSRX-)
- net U3RXDN4: now also U1.65 (U3RXDN4)
- net U3RXDP4: now reaches J2.6 (SSRX+)
- net U3RXDP4: now also U1.64 (U3RXDP4)
- net U3TXDN4: now reaches J2.8 (SSTX-)
- net U3TXDN4: now also C38.1
- net U3TXDP4: now reaches J2.9 (SSTX+)
- net U3TXDP4: now also C37.2
- net Earth: now reaches J2.S1 (SHIELD)
- net Earth: now also J2.S2 (SHIELD__1), J2.S3 (SHIELD__2), J2.S4 (SHIELD__3), J3.S1 (SHIELD), J3.S2 (SHIELD__1), J3.S3 (SHIELD__2), J3.S4 (SHIELD__3), J4.S1 (SHIELD), J4.S2 (SHIELD__1), J4.S3 (SHIELD__2), J4.S4 (SHIELD__3), J5.S1 (SHIELD), J5.S2 (SHIELD__1), J5.S3 (SHIELD__2), J5.S4 (SHIELD__3), R12.2, R13.2, R14.2, R15.2
- net PRSNT: now reaches J1.A1 (~{PRSNT1})
- net PRSNT: now also J1.B17 (~{PRSNT2})
- net +3V3_INT: now reaches J1.A10 (+3.3V)
- net +3V3_INT: now also J1.A9 (+3.3V), J1.B8 (+3.3V), C33.1, C34.1, R10.2, R11.2
- net +12V: now reaches J1.A2 (+12V)
- net +12V: now also J1.A3 (+12V), J1.B1 (+12V), J1.B2 (+12V), J1.B3 (+12V), C35.1, C36.1
- net at J1.A6 (JTAG3): now also J1.A7 (JTAG4)
- net +3V3_AUX: now reaches J1.B10 (3.3Vaux)
- net +3V3_AUX: now also TP3.1
- net at J4.1 (VBUS): now also FB4.2
- net U2DM2: now reaches J4.2 (D-)
- net U2DM2: now also U1.51 (U2DM2)
- net U2DP2: now reaches J4.3 (D+)
- net U2DP2: now also U1.50 (U2DP2)
- net U3RXDN2: now reaches J4.5 (SSRX-)
- net U3RXDN2: now also U1.48 (U3RXDN2)
- net U3RXDP2: now reaches J4.6 (SSRX+)
- net U3RXDP2: now also U1.47 (U3RXDP2)
- net U3TXDN2: now reaches J4.8 (SSTX-)
- net U3TXDN2: now also C42.1
- net U3TXDP2: now reaches J4.9 (SSTX+)
- net U3TXDP2: now also C41.2
- net OCI4B: now reaches U1.20 (OCI4B)
- net PPON4: now reaches U1.21 (PPON4)
- net OCI3B: now reaches U1.22 (OCI3B)
- net PPON3: now reaches U1.23 (PPON3)
- net OCI2B: now reaches U1.24 (OCI2B)
- net OCI2B: now also U1.26 (OCI1B)
- net PPON2: now reaches U1.25 (PPON2)
- net PPON1: now reaches U1.27 (PPON1)
- net U3TXDP1_H: now reaches U1.35 (U3TXDP1)
- net U3TXDP1_H: now also C43.1
- net U3TXDN1_H: now reaches U1.36 (U3TXDN1)
- net U3TXDN1_H: now also C44.2
- net U3RXDP1: now reaches U1.38 (U3RXDP1)
- net U3RXDP1: now also J5.6 (SSRX+)
- net U3RXDN1: now reaches U1.39 (U3RXDN1)
- net U3RXDN1: now also J5.5 (SSRX-)
- net U2DP1: now reaches U1.41 (U2DP1)
- net U2DP1: now also J5.3 (D+)
- net U2DM1: now reaches U1.42 (U2DM1)
- net U2DM1: now also J5.2 (D-)
- net U3TXDP2_H: now reaches U1.44 (U3TXDP2)
- net U3TXDP2_H: now also C41.1
- net U3TXDN2_H: now reaches U1.45 (U3TXDN2)
- net U3TXDN2_H: now also C42.2
- net U3TXDP3_H: now reaches U1.52 (U3TXDP3)
- net U3TXDP3_H: now also C39.1
- net U3TXDN3_H: now reaches U1.53 (U3TXDN3)
- net U3TXDN3_H: now also C40.2
- net U3RXDP3: now reaches U1.55 (U3RXDP3)
- net U3RXDP3: now also J3.6 (SSRX+)
- net U3RXDN3: now reaches U1.56 (U3RXDN3)
- net U3RXDN3: now also J3.5 (SSRX-)
- net U2DP3: now reaches U1.58 (U2DP3)
- net U2DP3: now also J3.3 (D+)
- net U2DM3: now reaches U1.59 (U2DM3)
- net U2DM3: now also J3.2 (D-)
- net U3TXDP4_H: now reaches U1.61 (U3TXDP4)
- net U3TXDP4_H: now also C37.1
- net U3TXDN4_H: now reaches U1.62 (U3TXDN4)
- net U3TXDN4_H: now also C38.2
- net at J5.1 (VBUS): now also FB5.2
- net U3TXDN1: now reaches J5.8 (SSTX-)
- net U3TXDN1: now also C44.1
- net U3TXDP1: now reaches J5.9 (SSTX+)
- net U3TXDP1: now also C43.2
- net at J3.1 (VBUS): now also FB3.2
- net U3TXDN3: now reaches J3.8 (SSTX-)
- net U3TXDN3: now also C40.1
- net U3TXDP3: now reaches J3.9 (SSTX+)
- net U3TXDP3: now also C39.2
- new net +3V3: R10.1, R11.1
- new net VCCCH1: FB5.1
- new net VCCCH2: FB4.1
- new net VCCCH3: FB3.1
- new net VCCCH4: FB2.1
- no-connect marks 0 -> 6
Other:
- moved on the sheet: C1, C10, C11, C12, C13, C14, C15, C16, C17, C18, C19, C2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

Commit message: Added power conversion circuits
Parts:
- removed C35: 10uF, Capacitor_SMD:C_0805_2012Metric_Pad1.18x1.45mm_HandSolder, symbol 0_Custom:CAP_0805_10uF_16V
- added C35: 10uF, Capacitor_SMD:C_1206_3216Metric_Pad1.33x1.80mm_HandSolder, symbol 0_Custom:CAP_1206_10uF_25V
Connections:
- net +12V: now also C35.1
- net GND: now also C35.2
Changed lines of the file:
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@@
+	)
+	(symbol
+		(lib_id "0_Custom:CAP_1206_10uF_25V")
+		(at 69.85 57.15 0)
+		(unit 1)
+		(body_style 1)
+		(exclude_from_sim no)
+		(in_bom yes)
+		(on_board yes)
+		(in_pos_files yes)
+		(dnp no)
+		(fields_autoplaced yes)
+		(property "Reference" "C35"
+			(at 72.39 55.8862 0)
+			(show_name no)
+			(do_not_autoplace no)
+			(effects
+				(font
+					(size 1.27 1.27)
+				)
+				(justify left)
+			)
+		)
+		(property "Value" "10uF"
+			(at 72.39 58.4262 0)
+			(show_name no)
+			(do_not_autoplace no)
+			(effects
+				(font
+					(size 1.27 1.27)
+				)
+				(justify left)
+			)
+		)
+		(property "Footprint" "Capacitor_SMD:C_1206_3216Metric_Pad1.33x1.80mm_HandSolder"
+			(at 69.85 57.15 0)
+			(hide yes)
+			(show_name no)
+			(do_not_autoplace no)
+			(effects
+				(font
+					(size 1.27 1.27)
+				)
+			)
+		)
+		(property "Datasheet" "https://mm.digikey.com/Volume0/opasdata/d220001/medias/docus/8942/490_Chip_Multilayer_CAT2021_MLCC.pdf"
+			(at 69.85 57.15 0)
+			(hide yes)
+			(show_name no)
+			(do_not_autoplace no)
+			(effects
+				(font
+					(size 1.27 1.27)
+				)
+			)
+		)
+		(property "Description" "10 µF ±10% 25V Ceramic Capacitor X5R 1206 (3216 Metric)"
+			(at 69.85 57.15 0)
+			(hide yes)
+			(show_name no)
+			(do_not_autoplace no)
+			(effects
+				(font
+					(size 1.27 1.27)
+				)
+			)
+		)
+		(property "Package" "1206"
+			(at 69.85 57.15 0)
+			(hide yes)
+			(show_name no)
+			(do_not_autoplace no)
+			(effects
+				(font
+					(size 1.27 1.27)
+				)
+			)
+		)
+		(property "Manufacturer" "MURATA"
+			(at 69.85 57.15 0)
+			(hide yes)
+			(show_name no)
+			(do_not_autoplace no)
+			(effects
+				(font
+					(size 1.27 1.27)
+				)
+			)
+		)
+		(property "Manufacturer Part #" "GRM319R61E106KA12D"
+			(at 69.85 57.15 0)
+			(hide yes)
+			(show_name no)
+			(do_not_autoplace no)
+			(effects
+				(font
+					(size 1.27 1.27)
+				)
+			)
+		)
+		(property "DigiKey Part #" "490-5525-1-ND"
+			(at 69.85 57.15 0)
+			(hide yes)
+			(show_name no)
+			(do_not_autoplace no)
+			(effects
+				(font
+					(size 1.27 1.27)
+				)
+			)
+		)
+		(property "LCSC Part #" "C162437"
+			(at 69.85 57.15 0)
+			(hide yes)
+			(show_name no)
+			(do_not_autoplace no)
+			(effects
+				(font
+					(size 1.27 1.27)
+				)
+			)
+		)
+		(property "Voltage Rating" "25V"
+			(at 69.85 57.15 0)
+			(hide yes)
+			(show_name no)
+			(do_not_autoplace no)
+			(effects
+				(font
+					(size 1.27 1.27)
+				)
+			)
+		)
+		(pin "2"
+		)
+		(pin "1"
+		)
+		(instances
+			(project "USB_PCIE_Board"
+				(path "/0b6a8cbe-8bf6-4e77-b3bd-c1d3e39e0e4a"
+					(reference "C35")
+					(unit 1)
+				)
+			)
+		)
 	)
 	(symbol
@@
 					(unit 1)
 				)
-			)
-		)
-	)
-	(symbol
-		(lib_id "0_Custom:CAP_0805_10uF_16V")
-		(at 69.85 57.15 0)
-		(unit 1)
-		(body_style 1)
-		(exclude_from_sim no)
-		(in_bom yes)
-		(on_board yes)
-		(in_pos_files yes)
-		(dnp no)
-		(fields_autoplaced yes)
-		(property "Reference" "C35"
-			(at 72.39 55.8862 0)
-			(show_name no)
-			(do_not_autoplace no)
-			(effects
-				(font
-					(size 1.27 1.27)
-				)
-				(justify left)
-			)
-		)
-		(property "Value" "10uF"
-			(at 72.39 58.4262 0)
-			(show_name no)
-			(do_not_autoplace no)
-			(effects
-				(font
-					(size 1.27 1.27)
-				)
-				(justify left)
-			)
-		)
-		(property "Footprint" "Capacitor_SMD:C_0805_2012Metric_Pad1.18x1.45mm_HandSolder"
-			(at 69.85 57.15 0)
-			(hide yes)
-			(show_name no)
-			(do_not_autoplace no)
-			(effects
-				(font
-					(size 1.27 1.27)
-				)
-			)
-		)
-		(property "Datasheet" "https://yageogroup.com/content/datasheet/asset/file/UPY-GPHC_X7R_6_3V-TO-250V"
-			(at 69.85 57.15 0)
-			(hide yes)
-			(show_name no)
-			(do_not_autoplace no)
-			(effects
-				(font
-					(size 1.27 1.27)
-				)
-			)
-		)
-		(property "Description" "10 µF ±10% 16V Ceramic Capacitor X7R 0805 (2012 Metric)"
-			(at 69.85 57.15 0)
-			(hide yes)
-			(show_name no)
-			(do_not_autoplace no)
-			(effects
-				(font
-					(size 1.27 1.27)
-				)
-			)
-		)
-		(property "Package" "0805"
-			(at 69.85 57.15 0)
-			(hide yes)
-			(show_name no)
-			(do_not_autoplace no)
-			(effects
-				(font
-					(size 1.27 1.27)
-				)
-			)
-		)
-		(property "Manufacturer" "YAGEO"
-			(at 69.85 57.15 0)
-			(hide yes)
-			(show_name no)
-			(do_not_autoplace no)
-			(effects
-				(font
-					(size 1.27 1.27)
-				)
-			)
-		)
-		(property "Manufacturer Part #" "CC0805KKX7R7BB106"
-			(at 69.85 57.15 0)
-			(hide yes)
-			(show_name no)
-			(do_not_autoplace no)
-			(effects
-				(font
-					(size 1.27 1.27)
-				)
-			)
-		)
-		(property "DigiKey Part #" "311-3501-1-ND"
-			(at 69.85 57.15 0)
-			(hide yes)
-			(show_name no)
-			(do_not_autoplace no)
-			(effects
-				(font
-					(size 1.27 1.27)
-				)
-			)
-		)
-		(property "LCSC Part #" "C326595"
-			(at 69.85 57.15 0)
-			(hide yes)
-			(show_name no)
-			(do_not_autoplace no)
-			(effects
-				(font
-					(size 1.27 1.27)
-				)
-			)
-		)
-		(property "Voltage Rating" "16V"
-			(at 69.85 57.15 0)
-			(hide yes)
-			(show_name no)
-			(do_not_autoplace no)
-			(effects
-				(font
-					(size 1.27 1.27)
-				)
-			)
-		)
-		(pin "2"
-		)
-		(pin "1"
-		)
-		(instances
-			(project "USB_PCIE_Board"
-				(path "/0b6a8cbe-8bf6-4e77-b3bd-c1d3e39e0e4a"
-					(reference "C35")
-					(unit 1)
-				)

Commit message: Fix changes suggested by Claude review; added schematic and netlist to document folder
Parts:
- added U12, U13, U14, U15: SP3011-06UTG, 0_Custom:SON14_SP3011-06UTG_LTF-M, symbol 0_Custom:SP3011-06UTG_ESD
Connections:
- net GND: now also U12.10, U12.5, U13.10, U13.5, U14.10, U14.5, U15.10, U15.5
- net OCI2B: no longer U1.26 (OCI1B)
- net U2DM1: now also U15.6, U15.9
- net U2DM2: now also U14.6, U14.9
- net U2DM3: now also U13.6, U13.9
- net U2DM4: now also U12.6, U12.9
- net U2DP1: now also U15.7, U15.8
- net U2DP2: now also U14.7, U14.8
- net U2DP3: now also U13.7, U13.8
- net U2DP4: now also U12.7, U12.8
- net U3RXDN1: now also U15.12, U15.3
- net U3RXDN2: now also U14.12, U14.3
- net U3RXDN3: now also U13.12, U13.3
- net U3RXDN4: now also U12.12, U12.3
- net U3RXDP1: now also U15.11, U15.4
- net U3RXDP2: now also U14.11, U14.4
- net U3RXDP3: now also U13.11, U13.4
- net U3RXDP4: now also U12.11, U12.4
- net U3TXDN1: now also U15.1, U15.14
- net U3TXDN2: now also U14.1, U14.14
- net U3TXDN3: now also U13.1, U13.14
- net U3TXDN4: now also U12.1, U12.14
- net U3TXDP1: now also U15.13, U15.2
- net U3TXDP2: now also U14.13, U14.2
- net U3TXDP3: now also U13.13, U13.2
- net U3TXDP4: now also U12.13, U12.2
- new net OCI1B: U1.26 (OCI1B)
Other:
- moved on the sheet: C29, C37, C38, C39, C40, C41, C42, C43, C44, FB2, FB3, FB4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

Commit message: Place all components except host chip decoupling caps and the crystal circuit.
Parts:
- J2, J3, J4, J5: value GSB4116341HR -> 0484050001; footprint 0_Custom:AMPHENOL_GSB4116341HR -> 0_Custom:USB3_A_Molex_48406-0001_Horizontal_Stacked; symbol 0_Custom:GSB4116341HR -> 0_Custom:0484050001_USB; DigiKey Part # GSB4116341HR-ND -> 0484050001-ND; LCSC Part # C3013502 -> C6376748; Manufacturer Amphenol -> MOLEX; Manufacturer Part # GSB4116341HR -> 0484050001
- U1: footprint 0_Custom:QFN68_8X8_REN-M -> 0_Custom:QFN68_8X8_REN-M_Hand_Soldering
- U2: footprint Package_SO:HSOP-8-1EP_3.9x4.9mm_P1.27mm_EP2.3x2.3mm -> 0_Custom:HSOP-8-1EP_3.9x4.9mm_P1.27mm_EP2.3x2.3mm
Connections:
- net Earth: now also J2.SH (SHIELD__2), J3.SH (SHIELD__2), J4.SH (SHIELD__2), J5.SH (SHIELD__2); no longer J2.S1 (SHIELD), J2.S2 (SHIELD__1), J2.S3 (SHIELD__2), J2.S4 (SHIELD__3), J3.S1 (SHIELD), J3.S2 (SHIELD__1), J3.S3 (SHIELD__2), J3.S4 (SHIELD__3), J4.S1 (SHIELD), J4.S2 (SHIELD__1), J4.S3 (SHIELD__2), J4.S4 (SHIELD__3), J5.S1 (SHIELD), J5.S2 (SHIELD__1), J5.S3 (SHIELD__2), J5.S4 (SHIELD__3)
- net PETXN_H renamed PETX_HN
- net PETXP_H renamed PETX_HP
- net U2DM1 renamed U2D1N
- net U2D1N: now also U15.7, U15.8; no longer U15.6, U15.9
- net U2DM2 renamed U2D2N
- net U2D2N: now also U14.7, U14.8; no longer U14.6, U14.9
- net U2DM3 renamed U2D3N
- net U2D3N: now also U13.7, U13.8; no longer U13.6, U13.9
- net U2DM4 renamed U2D4N
- net U2D4N: now also U12.7, U12.8; no longer U12.6, U12.9
- net U2DP1 renamed U2D1P
- net U2D1P: now also U15.6, U15.9; no longer U15.7, U15.8
- net U2DP2 renamed U2D2P
- net U2D2P: now also U14.6, U14.9; no longer U14.7, U14.8
- net U2DP3 renamed U2D3P
- net U2D3P: now also U13.6, U13.9; no longer U13.7, U13.8
- net U2DP4 renamed U2D4P
- net U2D4P: now also U12.6, U12.9; no longer U12.7, U12.8
- net U3RXDN1 renamed U3RXD1N
- net U3RXD1N: now also U15.11, U15.4; no longer U15.12, U15.3
- net U3RXDN2 renamed U3RXD2N
- net U3RXD2N: now also U14.11, U14.4; no longer U14.12, U14.3
- net U3RXDN3 renamed U3RXD3N
- net U3RXD3N: now also U13.11, U13.4; no longer U13.12, U13.3
- net U3RXDN4 renamed U3RXD4N
- net U3RXD4N: now also U12.11, U12.4; no longer U12.12, U12.3
- net U3RXDP1 renamed U3RXD1P
- net U3RXD1P: now also U15.12, U15.3; no longer U15.11, U15.4
- net U3RXDP2 renamed U3RXD2P
- net U3RXD2P: now also U14.12, U14.3; no longer U14.11, U14.4
- net U3RXDP3 renamed U3RXD3P
- net U3RXD3P: now also U13.12, U13.3; no longer U13.11, U13.4
- net U3RXDP4 renamed U3RXD4P
- net U3RXD4P: now also U12.12, U12.3; no longer U12.11, U12.4
- net U3TXDN1 renamed U3TXD1N
- net U3TXD1N: now also U15.13, U15.2; no longer U15.1, U15.14
- net U3TXDN1_H renamed U3TXD1_HN
- net U3TXDN2 renamed U3TXD2N
- net U3TXD2N: now also U14.13, U14.2; no longer U14.1, U14.14
- net U3TXDN2_H renamed U3TXD2_HN
- net U3TXDN3 renamed U3TXD3N
- net U3TXD3N: now also U13.13, U13.2; no longer U13.1, U13.14
- net U3TXDN3_H renamed U3TXD3_HN
- net U3TXDN4 renamed U3TXD4N
- net U3TXD4N: now also U12.13, U12.2; no longer U12.1, U12.14
- net U3TXDN4_H renamed U3TXD4_HN
- net U3TXDP1 renamed U3TXD1P
- net U3TXD1P: now also U15.1, U15.14; no longer U15.13, U15.2
- net U3TXDP1_H renamed U3TXD1_HP
- net U3TXDP2 renamed U3TXD2P
- net U3TXD2P: now also U14.1, U14.14; no longer U14.13, U14.2
- net U3TXDP2_H renamed U3TXD2_HP
- net U3TXDP3 renamed U3TXD3P
- net U3TXD3P: now also U13.1, U13.14; no longer U13.13, U13.2
- net U3TXDP3_H renamed U3TXD3_HP
- net U3TXDP4 renamed U3TXD4P
- net U3TXD4P: now also U12.1, U12.14; no longer U12.13, U12.2
- net U3TXDP4_H renamed U3TXD4_HP
Other:
- moved on the sheet: C26, C27, R1

Commit message: Complete first pass of routing all nets without DRC
Parts:
- U2: footprint 0_Custom:HSOP-8-1EP_3.9x4.9mm_P1.27mm_EP2.3x2.3mm -> 0_Custom:HSOP-8-1EP_3.9x4.9mm_P1.27mm_EP2.3x2.3mm_FLASH
Changed lines of the file:
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@@
 			)
 		)
-		(property "Footprint" "0_Custom:HSOP-8-1EP_3.9x4.9mm_P1.27mm_EP2.3x2.3mm"
+		(property "Footprint" "0_Custom:HSOP-8-1EP_3.9x4.9mm_P1.27mm_EP2.3x2.3mm_FLASH"
 			(at 105.41 243.84 0)
 			(hide yes)

Commit message: Add mounting hole symbols to schematic and continue PCB DRC cleanup
Sync schematic with the board by adding H1-H4 mounting holes, and
continue working through DRC violations (dangling vias, hole
clearance, footprint mismatches) on the PCB.
Parts:
- added H1, H2, H3, H4: MountingHole, MountingHole:MountingHole_3.2mm_M3, symbol Mechanical:MountingHole
