File: USB_PCIE_Board.kicad_sch (KiCad schematic)
At the start: 84 parts, among them J1 Bus_PCI_Express_x1, J2 0484050001, J3 0484050001, J4 0484050001, J5 0484050001, U1 UPD720201K8-711-BAC-A, U12 SP3011-06UTG, U13 SP3011-06UTG, U14 SP3011-06UTG, U15 SP3011-06UTG, U2 MX25L4006EM1I-12G, X1 CS14522-24M

Commit message: Correct U1 part number to UPD720201K8-701-BAC-A; fix silkscreen; add LCSC order BOM
Schematic symbol/value/datasheet now match the part actually ordered and
populated. Regenerated schematic PDF and added the final LCSC BOM CSV.

Co-Authored-By: Claude Sonnet 5 <noreply@anthropic.com>
Parts:
- U1: value UPD720201K8-711-BAC-A -> UPD720201K8-701-BAC-A; footprint 0_Custom:QFN68_8X8_REN-M_Hand_Soldering -> 0_Custom:QFN68_8X8_REN-M; symbol 0_Custom:UPD720201K8-711-BAC-A -> 0_Custom:UPD720201K8-701-BAC-A
Changed lines of the file:
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@@
 	)
 	(symbol
-		(lib_id "0_Custom:UPD720201K8-711-BAC-A")
+		(lib_id "0_Custom:UPD720201K8-701-BAC-A")
 		(at 229.87 165.1 0)
 		(unit 1)
@@
 			)
 		)
-		(property "Value" "UPD720201K8-711-BAC-A"
+		(property "Value" "UPD720201K8-701-BAC-A"
 			(at 306.9433 335.28 0)
 			(show_name no)
@@
 			)
 		)
-		(property "Footprint" "0_Custom:QFN68_8X8_REN-M_Hand_Soldering"
+		(property "Footprint" "0_Custom:QFN68_8X8_REN-M"
 			(at 229.87 165.1 0)
 			(hide yes)
@@
 			)
 		)
-		(property "Datasheet" "UPD720201K8-711-BAC-A"
+		(property "Datasheet" "https://www.renesas.com/us/en/document/dst/upd720201upd720202-datasheet?r=1260536"
 			(at 229.87 165.1 0)
 			(hide yes)
